Commit message: Robotino moves in Gazebo

File: rto_description/urdf/components/rto_body.urdf.xacro (robot description, xacro)
@@ -18,9 +18,9 @@
             </inertial>
             <visual>
-                <origin xyz="0.01 0 0" rpy="0 0 ${M_PI/2}"/>
-                <geometry>
-                    <mesh filename="package://rto_description/meshes/parts/rto_base.dae"
-                        scale="${M_SCALE} ${M_SCALE} ${M_SCALE}"/>
-                </geometry>
+            <origin xyz="0.01 0 0" rpy="0 0 ${M_PI/2}"/>
+            <geometry>
+                <mesh filename="file:///home/mike/robotino3/robotino3ros2/rto_description/meshes/parts/rto_base.dae"
+                    scale="${M_SCALE} ${M_SCALE} ${M_SCALE}"/>
+            </geometry>
             </visual>
             <collision>

File: rto_description/urdf/components/rto_parts.urdf.xacro (robot description, xacro)
@@ -12,14 +12,24 @@
         <link name="${name}_link">
             <inertial>
-                <mass value="0.00001"/>
-                <origin xyz="0 0 0"/>
-                <inertia ixx="1.0" ixy="0.0" ixz="0.0" iyy="1.0" iyz="0.0" izz="1.0"/>
+            <mass value="0.2"/>
+            <origin xyz="0 0 0"/>
+            <inertia
+                ixx="0.0001" ixy="0.0" ixz="0.0"
+                iyy="0.0001" iyz="0.0"
+                izz="0.0001"/>
             </inertial>
             <visual>
-                <origin xyz="0 0 0" rpy="0 0 0"/>
-                <geometry>
-                    <mesh filename="package://rto_description/meshes/parts/rto_wheel.dae" scale="${M_SCALE} ${M_SCALE} ${M_SCALE}"/>
-                </geometry>
+            <origin xyz="0 0 0" rpy="0 0 0"/>
+            <geometry>
+                <mesh filename="file:///home/mike/robotino3/robotino3ros2/rto_description/meshes/parts/rto_wheel.dae"
+                    scale="${M_SCALE} ${M_SCALE} ${M_SCALE}"/>
+            </geometry>
             </visual>
+            <collision>
+            <origin xyz="0 0 0" rpy="1.5708 0 0"/>
+            <geometry>
+                <cylinder radius="0.04" length="0.03"/>
+            </geometry>
+            </collision>
         </link>
         <gazebo reference="${name}_link">

File: rto_description/urdf/robots/rto-3.urdf.xacro (robot description, xacro)
@@ -6,18 +6,11 @@
   <xacro:include filename="$(find rto_description)/urdf/sensors/simple_lidar.urdf.xacro"/>
   <!-- <xacro:include filename="$(find rto_description)/urdf/sensors/hokuyo.urdf.xacro"/> -->
+ <!-- <xacro:include filename="$(find rto_description)/gazebo/robotino.gazebo"/> -->
   <xacro:rto_body/>
-  <!-- <xacro:plate parent="base_link" name="plate"/>
-  <xacro:bracket parent="base_link" name="bracket_hokuyo" scale="0.001">
-    <origin xyz="0.101 0 0.15" rpy="0 0 1.57"/>
-  </xacro:bracket> -->
   <!-- <xacro:bracket parent="base_link" name="bracket_camera" scale="0.000666666667">
     <origin xyz="0.084 0 0.271" rpy="0 3.14 1.57"/>
-  </xacro:bracket>
-  <xacro:sensor_asus_xtion_pro parent="base_link"/>
-  <xacro:hokuyo name="hokuyo" parent="base_link">
-    <origin xyz="0.08 0 0.2015" rpy="0 0 0"/>
-  </xacro:hokuyo> -->
+  </xacro:bracket>-->
   <xacro:simple_lidar name="lidar" parent="base_link">
-    <origin xyz="-0.03 0.0 0.24" rpy="0 0 0"/>
+    <origin xyz="-0.03 0.0 0.05" rpy="0 0 0"/>
   </xacro:simple_lidar>
 </robot>

File: rto_description/urdf/sensors/simple_lidar.urdf.xacro (robot description, xacro)
@@ -2,22 +2,27 @@
 <robot xmlns:xacro="http://wiki.ros.org/xacro">
   <xacro:macro name="simple_lidar" params="name parent *origin">
-    <link name="${name}_link">
+    <joint name="lidar_joint" type="fixed">
+      <parent link="base_link"/>
+      <child link="lidar_link"/>
+      <origin xyz="-0.03 0.0 0.24" rpy="0 0 0"/>
+    </joint>
+    <link name="lidar_link">
       <visual>
-        <origin xyz="0 0 0" rpy="0 0 0"/>
+        <origin xyz="0 0 0.025" rpy="0 0 0"/>
         <geometry>
-          <cylinder radius="0.04" length="0.05"/>
+          <cylinder length="0.05" radius="0.04"/>
         </geometry>
-        <material name="${name}_black">
-          <color rgba="0.01 0.01 0.01 1.0"/>
+        <material name="lidar_black">
+          <color rgba="0.0 0.0 0.0 1.0"/>
         </material>
       </visual>
       <collision>
-        <origin xyz="0 0 0" rpy="0 0 0"/>
+        <origin xyz="0 0 0.025" rpy="0 0 0"/>
         <geometry>
-          <cylinder radius="0.04" length="0.05"/>
+          <cylinder length="0.05" radius="0.04"/>
         </geometry>
       </collision>
       <inertial>
-        <origin xyz="0 0 0" rpy="0 0 0"/>
+        <origin xyz="0 0 0.025" rpy="0 0 0"/>
         <mass value="0.1"/>
         <inertia
@@ -27,9 +32,4 @@
       </inertial>
     </link>
-    <joint name="${name}_joint" type="fixed">
-      <parent link="${parent}"/>
-      <child link="${name}_link"/>
-      <xacro:insert_block name="origin"/>
-    </joint>
   </xacro:macro>
 </robot>

Commit message: Swithing to Gazebo Fortress

File: rto_description/urdf/components/rto_body.urdf.xacro (robot description, xacro)
@@ -18,9 +18,9 @@
             </inertial>
             <visual>
-            <origin xyz="0.01 0 0" rpy="0 0 ${M_PI/2}"/>
-            <geometry>
-                <mesh filename="file:///home/mike/robotino3/robotino3ros2/rto_description/meshes/parts/rto_base.dae"
-                    scale="${M_SCALE} ${M_SCALE} ${M_SCALE}"/>
-            </geometry>
+                <origin xyz="0.01 0 0" rpy="0 0 ${M_PI/2}"/>
+                <geometry>
+                    <mesh filename="package://rto_description/meshes/parts/rto_base.dae"
+                        scale="${M_SCALE} ${M_SCALE} ${M_SCALE}"/>
+                </geometry>
             </visual>
             <collision>

File: rto_description/urdf/robots/rto-3.urdf.xacro (robot description, xacro)
@@ -11,6 +11,6 @@
     <origin xyz="0.084 0 0.271" rpy="0 3.14 1.57"/>
   </xacro:bracket>-->
-  <xacro:simple_lidar name="lidar" parent="base_link">
-    <origin xyz="-0.03 0.0 0.05" rpy="0 0 0"/>
-  </xacro:simple_lidar>
+<xacro:simple_lidar name="lidar" parent="base_link">
+  <origin xyz="0.0 0.0 0.21" rpy="0 0 0"/>
+</xacro:simple_lidar>
 </robot>

File: rto_description/urdf/sensors/simple_lidar.urdf.xacro (robot description, xacro)
@@ -2,10 +2,10 @@
 <robot xmlns:xacro="http://wiki.ros.org/xacro">
   <xacro:macro name="simple_lidar" params="name parent *origin">
-    <joint name="lidar_joint" type="fixed">
-      <parent link="base_link"/>
-      <child link="lidar_link"/>
-      <origin xyz="-0.03 0.0 0.24" rpy="0 0 0"/>
+    <joint name="${name}_joint" type="fixed">
+      <parent link="${parent}"/>
+      <child link="${name}_link"/>
+      <xacro:insert_block name="origin"/>
     </joint>
-    <link name="lidar_link">
+    <link name="${name}_link">
       <visual>
         <origin xyz="0 0 0.025" rpy="0 0 0"/>
@@ -32,4 +32,39 @@
       </inertial>
     </link>
+    <gazebo reference="${name}_link">
+      <sensor name="${name}_gpu_lidar" type="gpu_lidar">
+        <pose>0 0 0.025 0 0 0</pose>
+        <topic>/lidar_scan</topic>
+        <update_rate>10</update_rate>
+        <always_on>true</always_on>
+        <visualize>true</visualize>
+        <ray>
+          <scan>
+            <horizontal>
+              <samples>360</samples>
+              <resolution>1</resolution>
+              <min_angle>-3.14159</min_angle>
+              <max_angle>3.14159</max_angle>
+            </horizontal>
+            <vertical>
+              <samples>1</samples>
+              <resolution>1</resolution>
+              <min_angle>0.0</min_angle>
+              <max_angle>0.0</max_angle>
+            </vertical>
+          </scan>
+          <range>
+            <min>0.12</min>
+            <max>6.0</max>
+            <resolution>0.01</resolution>
+          </range>
+          <noise>
+            <type>gaussian</type>
+            <mean>0.0</mean>
+            <stddev>0.01</stddev>
+          </noise>
+        </ray>
+      </sensor>
+    </gazebo>
   </xacro:macro>
 </robot>

Commit message: Potencial field implementation with bug

File: rto_description/urdf/components/rto_body.urdf.xacro (robot description, xacro)
@@ -56,13 +56,17 @@
         <!-- gazebo control -->
         <gazebo>
-            <plugin name="object_controller" filename="libgazebo_ros_planar_move.so">
-                <commandTopic>cmd_vel</commandTopic>
-                <odometryTopic>odom</odometryTopic>
-                <odometryFrame>odom</odometryFrame>
-                <odometryRate>20</odometryRate>
-                <robotBaseFrame>base_link</robotBaseFrame>
-                <publishTF>true</publishTF>
+            <plugin
+                filename="libignition-gazebo6-velocity-control-system.so"
+                name="ignition::gazebo::systems::VelocityControl">
+                <topic>/cmd_vel</topic>
             </plugin>
-            <plugin name="gazebo_ros_control" filename="libgazebo_ros_control.so"/>
+            <plugin
+                filename="libignition-gazebo6-odometry-publisher-system.so"
+                name="ignition::gazebo::systems::OdometryPublisher">
+                <odom_frame>odom</odom_frame>
+                <robot_base_frame>base_link</robot_base_frame>
+                <odom_topic>/odom</odom_topic>
+                <dimensions>2</dimensions>
+            </plugin>
         </gazebo>
     </xacro:macro>

File: rto_description/urdf/robots/rto-3.urdf.xacro (robot description, xacro)
@@ -11,6 +11,17 @@
     <origin xyz="0.084 0 0.271" rpy="0 3.14 1.57"/>
   </xacro:bracket>-->
-<xacro:simple_lidar name="lidar" parent="base_link">
-  <origin xyz="0.0 0.0 0.21" rpy="0 0 0"/>
-</xacro:simple_lidar>
+  <xacro:simple_lidar name="lidar" parent="base_link">
+    <origin xyz="0.0 0.0 0.21" rpy="0 0 0"/>
+  </xacro:simple_lidar>
+  <gazebo>
+    <plugin
+      filename="ignition-gazebo-odometry-publisher-system"
+      name="ignition::gazebo::systems::OdometryPublisher">
+      <odom_frame>odom</odom_frame>
+      <robot_base_frame>base_link</robot_base_frame>
+      <odom_publish_frequency>50</odom_publish_frequency>
+      <odom_topic>/odom</odom_topic>
+      <dimensions>2</dimensions>
+    </plugin>
+  </gazebo>
 </robot>

File: rto_description/urdf/sensors/simple_lidar.urdf.xacro (robot description, xacro)
@@ -38,5 +38,5 @@
         <update_rate>10</update_rate>
         <always_on>true</always_on>
-        <visualize>true</visualize>
+        <visualize>false</visualize>
         <ray>
           <scan>
