Commit message: URDF model in RVIZ

File: rto_description/urdf/robots/rto-3.urdf.xacro (robot description, xacro)
@@ -4,11 +4,12 @@
   <xacro:include filename="$(find rto_description)/urdf/components/rto_body.urdf.xacro"/>
   <xacro:include filename="$(find rto_description)/urdf/sensors/asus_xtion_pro.urdf.xacro"/>
-  <xacro:include filename="$(find rto_description)/urdf/sensors/hokuyo.urdf.xacro"/>
+  <xacro:include filename="$(find rto_description)/urdf/sensors/simple_lidar.urdf.xacro"/>
+  <!-- <xacro:include filename="$(find rto_description)/urdf/sensors/hokuyo.urdf.xacro"/> -->
   <xacro:rto_body/>
-  <xacro:plate parent="base_link" name="plate"/>
+  <!-- <xacro:plate parent="base_link" name="plate"/>
   <xacro:bracket parent="base_link" name="bracket_hokuyo" scale="0.001">
     <origin xyz="0.101 0 0.15" rpy="0 0 1.57"/>
-  </xacro:bracket>
-  <xacro:bracket parent="base_link" name="bracket_camera" scale="0.000666666667">
+  </xacro:bracket> -->
+  <!-- <xacro:bracket parent="base_link" name="bracket_camera" scale="0.000666666667">
     <origin xyz="0.084 0 0.271" rpy="0 3.14 1.57"/>
   </xacro:bracket>
@@ -16,4 +17,7 @@
   <xacro:hokuyo name="hokuyo" parent="base_link">
     <origin xyz="0.08 0 0.2015" rpy="0 0 0"/>
-  </xacro:hokuyo>
+  </xacro:hokuyo> -->
+  <xacro:simple_lidar name="lidar" parent="base_link">
+    <origin xyz="-0.03 0.0 0.24" rpy="0 0 0"/>
+  </xacro:simple_lidar>
 </robot>

Commit message: Added camera xacro model

File: rto_description/urdf/robots/rto-3.urdf.xacro (robot description, xacro)
@@ -5,4 +5,5 @@
   <xacro:include filename="$(find rto_description)/urdf/sensors/asus_xtion_pro.urdf.xacro"/>
   <xacro:include filename="$(find rto_description)/urdf/sensors/simple_lidar.urdf.xacro"/>
+  <xacro:include filename="$(find rto_description)/urdf/sensors/camera.urdf.xacro"/>
   <!-- <xacro:include filename="$(find rto_description)/urdf/sensors/hokuyo.urdf.xacro"/> -->
  <!-- <xacro:include filename="$(find rto_description)/gazebo/robotino.gazebo"/> -->
@@ -11,4 +12,7 @@
     <origin xyz="0.084 0 0.271" rpy="0 3.14 1.57"/>
   </xacro:bracket>-->
+  <xacro:camera parent="base_link" name="camera">
+    <origin xyz="0.05 0.0 0.17" rpy="0 0 ${M_PI/2}"/>
+  </xacro:camera>
   <xacro:simple_lidar name="lidar" parent="base_link">
     <origin xyz="0.0 0.0 0.21" rpy="0 0 0"/>

File: rto_description/urdf/sensors/camera.urdf.xacro (robot description, xacro)
@@ -1,27 +1,70 @@
 <?xml version="1.0"?>
-<robot name="sensor_camera" xmlns:xacro="http://wiki.ros.org/xacro">
+<robot xmlns:xacro="http://www.ros.org/wiki/xacro" name="logitech_c920_camera">
   <xacro:property name="M_PI" value="3.14159"/>
-  <xacro:property name="M_SCALE" value="0.01"/>
-  <xacro:macro name="camera" params="parent name *origin">
-    <joint name="${name}_joint" type="fixed">
-      <insert_block name="origin" />
+  <xacro:macro name="camera" params="name parent *origin">
+    <!-- Stem: vertical mount/clip -->
+    <joint name="${name}_mount_joint" type="fixed">
       <parent link="${parent}"/>
-      <child link="${name}_link" />
+      <child  link="${name}_mount_link"/>
+      <xacro:insert_block name="origin"/>
     </joint>
-    <link name="${name}_link">
+    <link name="${name}_mount_link">
+      <visual>
+        <origin xyz="0 0.03 0" rpy="0 0 ${M_PI/2}"/>
+        <geometry>
+          <box size="0.04 0.02 0.01"/>
+        </geometry>
+        <material name="camera_dark_grey">
+          <color rgba="0.0 0.0 0.0 1.0"/>
+        </material>
+      </visual>
+      <collision>
+        <origin xyz="0 0.03 0" rpy="0 0 ${M_PI/2}"/>
+          <box size="0.04 0.02 0.01"/>
+      </collision>
       <inertial>
-        <mass value="0.00001" />
-        <origin xyz="0 0 0" />
-        <inertia ixx="1.0" ixy="0.0" ixz="0.0"
-          iyy="1.0" iyz="0.0"
-          izz="1.0" />
+        <mass value="0.02"/>
+        <inertia ixx="1e-6" ixy="0" ixz="0"
+                 iyy="1e-6" iyz="0" izz="1e-6"/>
       </inertial>
+    </link>
+    <!-- Bar: horizontal lens body (top of the T) -->
+    <joint name="${name}_bar_joint" type="fixed">
+      <parent link="${name}_mount_link"/>
+      <child  link="${name}_bar_link"/>
+      <origin xyz="0 0 0.02" rpy="0 0 0"/>
+    </joint>
+    <link name="${name}_bar_link">
       <visual>
-        <origin xyz="0 0 0" rpy="0 0 0" />
+        <origin xyz="0 0 0" rpy="0 0 0"/>
         <geometry>
-          <mesh filename="package://rto_description/meshes/sensors/camera.dae" scale="${M_SCALE} ${M_SCALE} ${M_SCALE}"/>
+          <box size="0.08 0.03 0.03"/>
         </geometry>
+        <material name="camera_black">
+          <color rgba="0.0 0.0 0.0 1.0"/>
+        </material>
       </visual>
+      <collision>
+        <origin xyz="0 0 0" rpy="0 0 0"/>
+        <geometry>
+          <box size="0.08 0.03 0.03"/>
+        </geometry>
+      </collision>
+      <inertial>
+        <mass value="0.16"/>
+        <inertia ixx="1e-4" ixy="0" ixz="0"
+                iyy="1e-5" iyz="0" izz="1e-4"/>
+      </inertial>
     </link>
+    <!-- Optical frame -->
+    <joint name="${name}_optical_joint" type="fixed">
+      <parent link="${name}_bar_link"/>
+      <child  link="${name}_optical_frame"/>
+      <origin xyz="0 0 0.02" rpy="-1.5708 0 -1.5708"/>
+    </joint>
+    <link name="${name}_optical_frame"/>
+    <gazebo reference="${name}_bar_link">
+      <!-- add sensor plugin here if needed -->
+    </gazebo>
   </xacro:macro>
 </robot>
