Commit message: Added camera in gazebo

File: rto_description/urdf/sensors/camera.urdf.xacro (robot description, xacro)
@@ -1,10 +1,10 @@
 <?xml version="1.0"?>
 <robot xmlns:xacro="http://www.ros.org/wiki/xacro" name="logitech_c920_camera">
-  <xacro:property name="M_PI" value="3.14159"/>
+  <xacro:property name="M_PI" value="3.141592653589793"/>
   <xacro:macro name="camera" params="name parent *origin">
-    <!-- Stem: vertical mount/clip -->
+    <!-- Mount / stem -->
     <joint name="${name}_mount_joint" type="fixed">
       <parent link="${parent}"/>
-      <child  link="${name}_mount_link"/>
+      <child link="${name}_mount_link"/>
       <xacro:insert_block name="origin"/>
     </joint>
@@ -21,5 +21,7 @@
       <collision>
         <origin xyz="0 0.03 0" rpy="0 0 ${M_PI/2}"/>
+        <geometry>
           <box size="0.04 0.02 0.01"/>
+        </geometry>
       </collision>
       <inertial>
@@ -29,13 +31,13 @@
       </inertial>
     </link>
-    <!-- Bar: horizontal lens body (top of the T) -->
+    <!-- Camera body / horizontal bar -->
     <joint name="${name}_bar_joint" type="fixed">
       <parent link="${name}_mount_link"/>
-      <child  link="${name}_bar_link"/>
-      <origin xyz="0 0 0.02" rpy="0 0 0"/>
+      <child link="${name}_bar_link"/>
+      <origin xyz="0 0 0.02" rpy="0 0 -${M_PI/2}"/>
     </joint>
     <link name="${name}_bar_link">
       <visual>
-        <origin xyz="0 0 0" rpy="0 0 0"/>
+        <origin xyz="0 0 0" rpy="0 0 -${M_PI/2}"/>
         <geometry>
           <box size="0.08 0.03 0.03"/>
@@ -54,16 +56,44 @@
         <mass value="0.16"/>
         <inertia ixx="1e-4" ixy="0" ixz="0"
-                iyy="1e-5" iyz="0" izz="1e-4"/>
+                 iyy="1e-5" iyz="0" izz="1e-4"/>
       </inertial>
     </link>
-    <!-- Optical frame -->
+    <!-- ROS optical frame:
+         camera_bar_link:      x forward, y left, z up
+         camera_optical_frame: z forward, x right, y down
+    -->
     <joint name="${name}_optical_joint" type="fixed">
       <parent link="${name}_bar_link"/>
-      <child  link="${name}_optical_frame"/>
-      <origin xyz="0 0 0.02" rpy="-1.5708 0 -1.5708"/>
+      <child link="${name}_optical_frame"/>
+      <origin xyz="0 0 0" rpy="0 ${M_PI/2} 0"/>
     </joint>
     <link name="${name}_optical_frame"/>
+    <!-- Gazebo Sim camera sensor -->
     <gazebo reference="${name}_bar_link">
-      <!-- add sensor plugin here if needed -->
+      <sensor name="${name}_sensor" type="camera">
+        <always_on>true</always_on>
+        <update_rate>10</update_rate>
+        <visualize>true</visualize>
+        <!-- Gazebo Transport topic -->
+        <topic>/${name}/image_raw</topic>
+        <!-- Sensor pose relative to camera_bar_link -->
+        <pose>0 0 0 0 0 0</pose>
+        <!-- ROS/Gazebo frame information -->
+        <frame_id>${name}_optical_frame</frame_id>
+        <camera>
+          <horizontal_fov>1.089</horizontal_fov>
+          <!-- Important for camera_info -->
+          <optical_frame_id>${name}_optical_frame</optical_frame_id>
+          <image>
+            <width>640</width>
+            <height>480</height>
+            <format>R8G8B8</format>
+          </image>
+          <clip>
+            <near>0.05</near>
+            <far>8.0</far>
+          </clip>
+        </camera>
+      </sensor>
     </gazebo>
   </xacro:macro>
