Commit message: Correct config for 0.25x0.25m Tags

File: rto_description/urdf/sensors/camera.urdf.xacro (robot description, xacro)
@@ -66,5 +66,5 @@
       <parent link="${name}_bar_link"/>
       <child link="${name}_optical_frame"/>
-      <origin xyz="0 0 0" rpy="0 ${M_PI/2} 0"/>
+      <origin xyz="0 0 0" rpy="${3 * M_PI/2} 0 ${3 * M_PI/2}"/>
     </joint>
     <link name="${name}_optical_frame"/>
